Commit message: Fix Astribot black scene: replace GLB/OBJ mesh visuals with primitives
Gazebo Classic (OGRE) cannot parse .glb or .gltf mesh files. The Astribot
base URDF referenced 21 mesh files (20 .glb + 1 non-existent .obj), causing
cascading mesh-load failures that left the OGRE renderer in a broken state
and produced a completely black scene — even the world/ground didn't render.

Fix: replace every <visual><mesh .glb|.obj/> with simple geometric primitives
(cylinders, spheres, boxes) reused from each link's collision geometry.
The robot now renders as simple grey shapes in Gazebo, matching the quality
of other simulation-only models.

Also removed the outdated "only the 3D visual is missing" comment from README.

Co-Authored-By: Claude Sonnet 4.6 <noreply@anthropic.com>

File: src/astribot_description/urdf/astribot_s1_base.urdf (robot description, URDF)
Before this commit: robot astribot_s1, 21 links, 20 joints
Links:
- link base_link: geometry collision cylinder length=0.1 radius=0.3; visual cylinder length=0.1 radius=0.3
- link head_link_1: geometry visual box size=0.1 0.1 0.1
- link head_link_2: geometry collision sphere radius=0.11; visual sphere radius=0.11
- link left_link_1: geometry visual box size=0.1 0.1 0.1
- link left_link_2: geometry visual box size=0.1 0.1 0.1
- link left_link_3: geometry collision cylinder length=0.18 radius=0.05; visual cylinder length=0.18 radius=0.05
- link left_link_4: geometry collision sphere radius=0.06; visual sphere radius=0.06
- link left_link_5: geometry collision cylinder length=0.14 radius=0.05; visual cylinder length=0.14 radius=0.05
- link left_link_6: geometry visual box size=0.1 0.1 0.1
- link left_link_7: geometry collision sphere radius=0.05; visual sphere radius=0.05
- link right_link_1: geometry visual box size=0.1 0.1 0.1
- link right_link_2: geometry visual box size=0.1 0.1 0.1
- link right_link_3: geometry collision cylinder length=0.18 radius=0.05; visual cylinder length=0.18 radius=0.05
- link right_link_4: geometry collision sphere radius=0.06; visual sphere radius=0.06
- link right_link_5: geometry collision cylinder length=0.14 radius=0.05; visual cylinder length=0.14 radius=0.05
- link right_link_6: geometry visual box size=0.1 0.1 0.1
- link right_link_7: geometry collision sphere radius=0.05; visual sphere radius=0.05
- link torso_link_1: geometry collision cylinder length=0.3 radius=0.1; visual cylinder length=0.3 radius=0.1
- link torso_link_2: geometry collision cylinder length=0.3 radius=0.1; visual cylinder length=0.3 radius=0.1
- link torso_link_3: geometry collision cylinder length=0.35 radius=0.09; visual cylinder length=0.35 radius=0.09
- link torso_link_4: geometry visual box size=0.1 0.1 0.1
